File: kicad/cacophonator.kicad_sch (KiCad schematic)
At the start: 40 parts, among them J1 AUDIO OUTPUT, SW1 POWER, SW2 CHARGE, U1 40106

Commit message: v1
Parts:
- removed R9: 100k, Resistor_THT:R_Axial_DIN0204_L3.6mm_D1.6mm_P5.08mm_Horizontal, symbol Device:R_Small
- removed RV1, RV2, RV3, RV4, RV6, RV7: 1M, Connector_Molex:Molex_KK-254_AE-6410-03A_1x03_P2.54mm_Vertical, symbol Device:R_Potentiometer
- removed RV5: 10k, Connector_Molex:Molex_KK-254_AE-6410-03A_1x03_P2.54mm_Vertical, symbol Device:R_Potentiometer
- added D3, D4: 1N4004*, Diode_THT:D_DO-35_SOD27_P7.62mm_Horizontal, symbol Device:D_Small_Filled
- added H1, H10, H2, H3, H4, H5, H6, H7, H8, H9: MountingHole, MountingHole:MountingHole_3.2mm_M3_ISO7380_Pad, symbol Mechanical:MountingHole
- added J1: Jack-DC, Connector_JST:JST_PH_B2B-PH-K_1x02_P2.00mm_Vertical, symbol Connector:Jack-DC
- added RV1, RV2, RV3, RV4, RV5, RV6: 1M, Connector_JST:JST_PH_B2B-PH-K_1x02_P2.00mm_Vertical, symbol Device:R_Variable
- added RV7: 10k, Connector_JST:JST_PH_B2B-PH-K_1x02_P2.00mm_Vertical, symbol Device:R_Variable
- added RV8: 100k log, Connector_JST:JST_PH_B3B-PH-K_1x03_P2.00mm_Vertical, symbol Device:R_Potentiometer
- BT1, SW1, SW2: footprint Connector_Molex:Molex_KK-254_AE-6410-02A_1x02_P2.54mm_Vertical -> Connector_JST:JST_PH_B2B-PH-K_1x02_P2.00mm_Vertical
- C11, C9: value 2200uF -> 22uF
- C7: footprint Capacitor_THT:CP_Radial_D7.5mm_P2.50mm -> Capacitor_THT:CP_Radial_D10.0mm_P5.00mm
- D2: footprint LED_THT:LED_D5.0mm -> Connector_JST:JST_PH_B2B-PH-K_1x02_P2.00mm_Vertical
- J2: renamed from J1; footprint Connector_Molex:Molex_KK-254_AE-6410-02A_1x02_P2.54mm_Vertical -> Connector_JST:JST_PH_B2B-PH-K_1x02_P2.00mm_Vertical
Connections:
- net GND: now also C10.2, C11.2, C8.2, C9.2, J1.2, RV8.3; no longer C10.1, C11.1, C8.1, C9.1
- net VCC: now also R10.1, SW1.2 (B), SW2.2; no longer BT1.1 (+), SW1.1 (A), SW2.1
- net at C6.2: now also RV8.1; no longer J2.1 (In)
- net at R12.1: now also C9.1; no longer C9.2
- net at R12.2, U1.10: now also RV5.1
- net at R13.1, U1.13: now also C10.1; no longer C10.2
- net at R13.2: now also RV6.1
- net at R3.2: now also RV3.1
- net at R2.2: now also RV2.1
- net at R11.1, U1.11: now also C8.1; no longer C8.2
- net at R11.2: now also RV5.2
- net at R8.2, U1.8: now also RV4.2
- net at R14.1: now also C11.1; no longer C11.2
- net at R14.2, U1.12: now also RV6.2
- net at R5.2, U1.2: now also RV1.2
- net at R4.2: now also RV4.1
- net at R6.2, U1.4: now also RV2.2
- net at C7.1, D1.1 (K), R10.2: now also RV7.2
- net at C5.1, U1.14 (VDD): now also RV7.1
- net at R7.2, U1.6: now also RV3.2
- net at R1.2: now also RV1.1
- new net: D3.1 (K), D4.1 (K), SW1.1 (A), SW2.1
- new net: D3.2 (A), J1.1
- new net: BT1.1 (+), D4.2 (A)
- new net: J2.1 (In), RV8.2
Other:
- note added: "10nF"
- note added: "2.2nF"
- note added: "DC IN *"
- note added: "Ideally Hi-Z no current"
- note added: "Makes no sense to use reverse diode if using diodes to mix power supplies"
- note added: "Notes: - Volume pot [Added] - Optional DC IN jack [Added] -"
- note added: "POWER & STARVE Control - Diode D1 is for reverse polarity"
- note added: "Resistive Mixer"
- note added: "Volume"
- note added: "keep extra space in PCB"
- note removed: "Notes: - Volume pot ?! - Output buffer ?"
- note removed: "POWER & STARVE Control - Diode is for reverse polarity"
- title: CACOPHONATOR 1.0 -> CACOPHONATOR 1.1
- moved on the sheet: BT1, C1, C10, C11, C2, C3, C4, C5, C7, C8, C9, D1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

Commit message: Minor updates
Other:
- note added: "Makes no sense to use reverse diode if using diodes to mix power supplies --- It can be used to add a discharge resistor that is added in-circuit via pushbutton"
- note removed: "Makes no sense to use reverse diode if using diodes to mix power supplies"
Changed lines of the file:
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@@
 		)
 	)
-	(text "Makes no sense to use\nreverse diode if using \ndiodes to mix power supplies"
+	(text "Makes no sense to use\nreverse diode if using \ndiodes to mix power supplies\n---\nIt can be used to add a discharge\nresistor that is added in-circuit\nvia pushbutton"
 		(exclude_from_sim no)
-		(at 107.95 161.036 0)
+		(at 108.204 165.862 0)
 		(effects
 			(font

Commit message: Added info to schematic
Other:
- note added: "Oscillators ----------- Frequency is inversely proportional to feedback resistance. When RV = 0 we sould have the highest frequency. Important tip for potentiometer soldering on the chassis."
Changed lines of the file:
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@@
+	)
+	(rectangle
+		(start 176.276 133.35)
+		(end 242.316 152.4)
+		(stroke
+			(width 0)
+			(type default)
+		)
+		(fill
+			(type none)
+		)
 	)
 	(rectangle
@@
 		)
 	)
+	(text "Oscillators\n-----------\n\nFrequency is inversely proportional to feedback resistance.\nWhen RV = 0 we sould have the highest frequency.\n\nImportant tip for potentiometer soldering on the chassis."
+		(exclude_from_sim no)
+		(at 208.28 142.24 0)
+		(effects
+			(font
+				(size 1.27 1.27)
+			)
+		)
+	)
